File: USB UART converter.kicad_pcb (KiCad board)
At the start: 2 copper layers, 32.5 x 14 mm, 19 parts, among them J1 USB_C_Receptacle_USB2.0_16P, J2 Conn_01x05_Pin, U1 CP2102N-Axx-xQFN28

Commit message: Adjusted the Diff pair and created the gnd plane
Parts:
- moved D2 4.72 mm to (59.5, 58.5)
- moved R2 1.58 mm to (59.0, 60.0)
- moved D3 1.50 mm to (59.5, 61.5)
Routing:
- net GND: track 45.3 -> 50.4 mm
- net /DP: track 15.8 -> 19.5 mm
- net /VBUS: track 43.1 -> 44.5 mm
- net /DN: track 17.9 -> 19.3 mm
- added copper zone on B.Cu, net GND
- added copper zone on F.Cu, net GND
