File: USB UART converter.kicad_sch (KiCad schematic)
At the start: 19 parts, among them J1 USB_C_Receptacle_USB2.0_16P, J2 Conn_01x05_Pin, U1 CP2102N-Axx-xQFN28

Commit message: Adjusted the Diff pair and created the gnd plane
Changed lines of the file:
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@@
 	(wire
 		(pts
-			(xy 45.72 124.46) (xy 45.72 127)
-		)
-		(stroke
-			(width 0)
-			(type default)
-		)
-	)
-	(wire
-		(pts
 			(xy 245.11 58.42) (xy 245.11 45.72)
 		)
@@
 	(wire
 		(pts
-			(xy 45.72 124.46) (xy 59.69 124.46)
+			(xy 57.15 50.8) (xy 63.5 50.8)
 		)
 		(stroke
@@
 	(wire
 		(pts
-			(xy 57.15 50.8) (xy 63.5 50.8)
+			(xy 73.66 38.1) (xy 57.15 38.1)
 		)
 		(stroke
@@
 	(wire
 		(pts
-			(xy 73.66 38.1) (xy 57.15 38.1)
+			(xy 46.99 124.46) (xy 46.99 137.16)
 		)
 		(stroke
@@
 	(wire
 		(pts
+			(xy 46.99 124.46) (xy 59.69 124.46)
+		)
+		(stroke
+			(width 0)
+			(type default)
+		)
+	)
+	(wire
+		(pts
 			(xy 34.29 80.01) (xy 41.91 80.01)
 		)
@@
 	(symbol
 		(lib_id "power:GND")
-		(at 45.72 127 0)
+		(at 46.99 137.16 0)
 		(unit 1)
 		(body_style 1)
@@
 		(fields_autoplaced yes)
 		(property "Reference" "#PWR06"
-			(at 45.72 133.35 0)
+			(at 46.99 143.51 0)
 			(hide yes)
 			(show_name no)
@@
 		)
 		(property "Value" "GND"
-			(at 45.72 132.08 0)
+			(at 46.99 142.24 0)
 			(show_name no)
 			(do_not_autoplace no)
@@
 		)
 		(property "Footprint" ""
-			(at 45.72 127 0)
+			(at 46.99 137.16 0)
 			(hide yes)
 			(show_name no)
@@
 		)
 		(property "Datasheet" ""
-			(at 45.72 127 0)
+			(at 46.99 137.16 0)
 			(hide yes)
 			(show_name no)
@@
 		)
 		(property "Description" "Power symbol creates a global label with name \"GND\" , ground"
-			(at 45.72 127 0)
+			(at 46.99 137.16 0)
 			(hide yes)
 			(show_name no)
